File: zero-percent-keyboard.kicad_pcb (KiCad board)
At the start: 2 copper layers, 197 parts, among them J1 USB4085-GF-A_REVA, SW1 SW_PUSH, U1 ATMEGA32U4, X1 XTAL_GND

Commit message: Progress
Parts:
- C1, C2, C3, C4, C5, C6, C7, C8, F1, R1, R2, R3, R4, R5, R6, SW1, U1, X1: moved to B.Cu
- moved F1 343.2 mm to (308.6, 6.48)
- moved R2 333.5 mm to (281.9, 27.8), turned to 90 degrees
- moved R3 326.9 mm to (279.9, 27.8), turned to 90 degrees
- moved R5 321.5 mm to (284.0, 27.8), turned to 90 degrees
- moved R4 320.2 mm to (277.9, 27.8), turned to 90 degrees
- moved J1 316.6 mm to (280.9, 20.7), turned to 180 degrees
- moved C7 243.6 mm to (192.9, 128.1), turned to 180 degrees
- moved C8 236.0 mm to (188.1, 133.2), turned to 270 degrees
- moved C6 232.1 mm to (182.7, 117.9), turned to 315 degrees
- moved X1 218.8 mm to (192.0, 131.7), turned to 180 degrees
- moved C2 205.4 mm to (176.1, 135.3), turned to 180 degrees
- moved C5 204.2 mm to (189.8, 126.3), turned to 45 degrees
- moved C1 203.3 mm to (186.5, 121.7), turned to 315 degrees
- moved U1 202.8 mm to (180.2, 127.0), turned to 225 degrees
- moved R6 202.5 mm to (151.1, 179.7)
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Connections:
- X1 pad 2: XTAL2 -> GND
- X1 pad 3: GND -> XTAL2
- X1 pad 4: (no net) -> GND
Routing:
- net D+: track 0.00 -> 176.9 mm, vias 0 -> 2
- net D-: track 0.00 -> 175.3 mm
- net XTAL1: track 0.00 -> 16.8 mm
- net +5V: track 0.00 -> 11.8 mm, vias 0 -> 2
- net Net-(J1-PadB5): track 0.00 -> 10.2 mm, vias 0 -> 1
- net GND: track 0.00 -> 8.98 mm
- net VCC: track 0.00 -> 8.14 mm
- net XTAL2: track 0.00 -> 6.96 mm
- net Net-(J1-PadA6): track 0.00 -> 4.72 mm
- net Net-(J1-PadA7): track 0.00 -> 4.52 mm, vias 0 -> 1
- net Net-(R1-Pad1): track 0.00 -> 2.17 mm
Other:
- board outline added: 324.1 x 118.4 mm
- net class Default: trace_width 0.25 -> 0.254
- net class Power added: clearance 0.2, trace_width 0.381, via_dia 0.8, via_drill 0.4
