File: zero-percent-keyboard.kicad_pcb (KiCad board)
At the start: 2 copper layers, 324.1 x 118.4 mm, 197 parts, among them J1 USB4085-GF-A_REVA, SW1 SW_PUSH, U1 ATMEGA32U4, X1 XTAL_GND

Commit message: Route traces
Routing:
- net ROW2: track 0.00 -> 336.6 mm, vias 0 -> 2
- net ROW3: track 0.00 -> 332.9 mm, vias 0 -> 2
- net ROW4: track 0.00 -> 17.1 mm

Commit message: Route traces
Routing:
- net ROW5: track 0.00 -> 331.6 mm
- net ROW4: track 17.1 -> 348.4 mm, vias 0 -> 2
- net Net-(D71-Pad2): track 0.00 -> 11.2 mm
- net Net-(D34-Pad2): track 0.00 -> 11.2 mm
- net Net-(D86-Pad2): track 0.00 -> 11.0 mm
- net Net-(D88-Pad2): track 0.00 -> 11.0 mm
- net Net-(D87-Pad2): track 0.00 -> 11.0 mm
- net Net-(D77-Pad2): track 0.00 -> 11.0 mm
- net Net-(D80-Pad2): track 0.00 -> 10.9 mm
- net Net-(D64-Pad2): track 0.00 -> 10.9 mm
- net Net-(D1-Pad2): track 0.00 -> 10.9 mm
- net Net-(D85-Pad2): track 0.00 -> 10.9 mm
- net Net-(D76-Pad2): track 0.00 -> 10.8 mm
- net Net-(D29-Pad2): track 0.00 -> 10.8 mm
- net Net-(D9-Pad2): track 0.00 -> 10.8 mm
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
Commit message: Progress
Routing:
- net COL1: track 0.00 -> 118.3 mm
- net COL9: track 0.00 -> 116.3 mm
- net COL10: track 0.00 -> 116.1 mm
- net COL2: track 0.00 -> 115.6 mm
- net COL12: track 0.00 -> 112.5 mm
- net COL11: track 0.00 -> 112.0 mm
- net COL5: track 0.00 -> 109.0 mm
- net COL13: track 0.00 -> 106.9 mm
- net COL0: track 0.00 -> 104.3 mm
- net COL15: track 0.00 -> 95.2 mm
- net COL14: track 0.00 -> 95.2 mm
- net COL6: track 0.00 -> 89.7 mm
- net COL8: track 0.00 -> 89.4 mm
- net COL7: track 0.00 -> 88.4 mm
- net COL4: track 0.00 -> 87.3 mm
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