File: _autosave-zero-percent-keyboard.kicad_pcb (KiCad board)
At the start: 2 copper layers, 324.1 x 118.4 mm, 197 parts, among them J1 USB4085-GF-A_REVA, SW1 SW_PUSH, U1 ATMEGA32U4, X1 XTAL_GND

Commit message: Route traces
Routing:
- net ROW2: track 0.00 -> 62.1 mm, vias 0 -> 2
Changed lines of the file:
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@@
     (thickness 1.6)
     (drawings 18)
-    (tracks 260)
+    (tracks 266)
     (zones 0)
     (modules 197)
@@
   (segment (start 32.512 56.896) (end 32.512 58.039) (width 0.254) (layer B.Cu) (net 24))
   (segment (start 32.512 58.039) (end 31.877 58.674) (width 0.254) (layer B.Cu) (net 24))
+  (segment (start 337.184 75.946) (end 337.184 77.09) (width 0.254) (layer B.Cu) (net 41))
+  (segment (start 337.184 77.09) (end 336.55 77.724) (width 0.254) (layer B.Cu) (net 41))
+  (via (at 279.4 77.724) (size 0.8) (drill 0.4) (layers F.Cu B.Cu) (net 41))
+  (segment (start 336.55 77.724) (end 279.527 77.724) (width 0.254) (layer B.Cu) (net 41))
+  (via (at 276.352 77.724) (size 0.8) (drill 0.4) (layers F.Cu B.Cu) (net 41))
+  (segment (start 279.4 77.724) (end 276.352 77.724) (width 0.254) (layer F.Cu) (net 41))
   (segment (start 278.792 24.68) (end 278.792 23.268) (width 0.381) (layer B.Cu) (net 100))
   (segment (start 278.792 23.33) (end 278.792 22.887) (width 0.381) (layer B.Cu) (net 100))
